File: remora.kicad_sch (KiCad schematic)
At the start: 74 parts, among them J1 ST_01x03, J2 ST_01x02, J3 ST_01x02, J4 ST_01x02, J5 ST_01x02, J6 ST_01x02, J7 Conn_01x05_Pin, J9 ST_01x02, K1 G5Q-1, Q1 MMBT2222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

Commit message: Add Switch
Parts:
- added SW1: SW_Push, Button_Switch_SMD:SW_Push_1P1T_NO_6x6mm_H9.5mm, symbol Switch:SW_Push
- R18: Mouser# 603-RC0805FR-073K3L -> 603-CFR-50JR-52-220R
- R21, R22, R24: Mouser# 603-CFR-50JR-52-220R -> 603-RC0805FR-073K3L
Connections:
- net GND: now also SW1.2
- net at U16.5 (IO12/TDI): now also SW1.1
- no-connect marks 24 -> 23
Changed lines of the file:
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@@
   (no_connect (at 254 52.705))
   (no_connect (at 254 50.165))
-  (no_connect (at 254 47.625))
   (no_connect (at 254 40.005))
   (no_connect (at 27.94 123.825))
@@
     (stroke (width 0) (type default))
   )
+  (wire (pts (xy 262.255 54.61) (xy 267.335 54.61))
+    (stroke (width 0) (type default))
+  )
   (wire (pts (xy 45.72 97.155) (xy 54.61 97.155))
     (stroke (width 0) (type default))
@@
     (stroke (width 0) (type default))
   )
+  (wire (pts (xy 277.495 54.61) (xy 277.495 56.515))
+    (stroke (width 0) (type default))
+  )
   (wire (pts (xy 67.945 41.91) (xy 67.945 41.275))
     (stroke (width 0) (type default))
@@
     (stroke (width 0) (type default))
   )
+  (wire (pts (xy 254 47.625) (xy 262.255 47.625))
+    (stroke (width 0) (type default))
+  )
   (wire (pts (xy 258.445 135.255) (xy 260.985 135.255))
     (stroke (width 0) (type default))
@@
     (stroke (width 0) (type default))
   )
+  (wire (pts (xy 262.255 47.625) (xy 262.255 54.61))
+    (stroke (width 0) (type default))
+  )
   (wire (pts (xy 169.545 139.065) (xy 182.88 139.065))
     (stroke (width 0) (type default))
@@
       (effects (font (size 1.27 1.27)) hide)
     )
-    (property "Mouser#" "603-CFR-50JR-52-220R" (at 260.985 140.97 0)
+    (property "Mouser#" "603-RC0805FR-073K3L" (at 260.985 140.97 0)
       (effects (font (size 1.27 1.27)) hide)
     )
@@
       (effects (font (size 1.27 1.27)) hide)
     )
-    (property "Mouser#" "603-RC0805FR-073K3L" (at 53.975 69.85 0)
+    (property "Mouser#" "603-CFR-50JR-52-220R" (at 53.975 69.85 0)
       (effects (font (size 1.27 1.27)) hide)
     )
@@
     )
   )
+  (symbol (lib_id "power:GND") (at 277.495 56.515 0) (unit 1)
+    (in_bom yes) (on_board yes) (dnp no) (fields_autoplaced)
+    (property "Reference" "#PWR04" (at 277.495 62.865 0)
+      (effects (font (size 1.27 1.27)) hide)
+    )
+    (property "Value" "GND" (at 277.495 61.595 0)
+      (effects (font (size 1.27 1.27)))
+    )
+    (property "Footprint" "" (at 277.495 56.515 0)
+      (effects (font (size 1.27 1.27)) hide)
+    )
+    (property "Datasheet" "" (at 277.495 56.515 0)
+      (effects (font (size 1.27 1.27)) hide)
+    )
+    (pin "1")
+    (instances
+      (project "remora"
+        (path "/cb2f202c-2f0c-437b-a702-06609217e330"
+          (reference "#PWR04") (unit 1)
+        )
+      )
+    )
+  )
   (symbol (lib_id "Device:R") (at 112.395 140.335 270) (unit 1)
     (in_bom yes) (on_board yes) (dnp no)
@@
       (effects (font (size 1.27 1.27)) hide)
     )
-    (property "Mouser#" "603-CFR-50JR-52-220R" (at 276.86 93.98 0)
+    (property "Mouser#" "603-RC0805FR-073K3L" (at 276.86 93.98 0)
       (effects (font (size 1.27 1.27)) hide)
     )
@@
     )
   )
+  (symbol (lib_id "Switch:SW_Push") (at 272.415 54.61 0) (unit 1)
+    (in_bom yes) (on_board yes) (dnp no) (fields_autoplaced)
+    (property "Reference" "SW1" (at 272.415 47.5447 0)
+      (effects (font (size 1.27 1.27)))
+    )
+    (property "Value" "SW_Push" (at 272.415 49.9689 0)
+      (effects (font (size 1.27 1.27)))
+    )
+    (property "Footprint" "Button_Switch_SMD:SW_Push_1P1T_NO_6x6mm_H9.5mm" (at 272.415 49.53 0)
+      (effects (font (size 1.27 1.27)) hide)
+    )
+    (property "Datasheet" "~" (at 272.415 49.53 0)
+      (effects (font (size 1.27 1.27)) hide)
+    )
+    (pin "2")
+    (pin "1")
+    (instances
+      (project "remora"
+        (path "/cb2f202c-2f0c-437b-a702-06609217e330"
+          (reference "SW1") (unit 1)
+        )
+      )
+    )
+  )
   (symbol (lib_id "Device:R") (at 273.05 93.98 180) (unit 1)
     (in_bom yes) (on_board yes) (dnp no)
@@
       (effects (font (size 1.27 1.27)) hide)
     )
-    (property "Mouser#" "603-CFR-50JR-52-220R" (at 273.05 93.98 0)
+    (property "Mouser#" "603-RC0805FR-073K3L" (at 273.05 93.98 0)
       (effects (font (size 1.27 1.27)) hide)
     )

Commit message: Modif commande v2.0
Parts:
- C3: footprint Capacitor_THT:C_Rect_L10.0mm_W4.0mm_P7.50mm_MKS4 -> Capacitor_THT:C_Rect_L11.5mm_W5.6mm_P10.00mm_MKT; LCSC# C2895620 -> C506867; Mouser# 667-ECW-FD2J104K4 -> (none)
- SW1: LCSC# (none) -> C255812; Mouser# (none) -> 179-TS046655BK160SMT
Connections:
- net at U16.16 (IO16): now also SW1.1
- net at U16.5 (IO12/TDI): no longer SW1.1
Changed lines of the file:
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@@
   (no_connect (at 213.36 71.755))
   (no_connect (at 213.36 64.135))
-  (no_connect (at 254 57.785))
+  (no_connect (at 254 47.625))
   (no_connect (at 254 90.805))
   (no_connect (at 213.36 69.215))
@@
     (stroke (width 0) (type dash))
   )
+  (wire (pts (xy 254 57.785) (xy 256.54 57.785))
+    (stroke (width 0) (type default))
+  )
   (wire (pts (xy 231.14 28.575) (xy 231.14 31.115))
     (stroke (width 0) (type default))
@@
     (stroke (width 0) (type dash))
   )
+  (wire (pts (xy 256.54 57.785) (xy 256.54 54.61))
+    (stroke (width 0) (type default))
+  )
   (wire (pts (xy 63.5 123.825) (xy 70.485 123.825))
     (stroke (width 0) (type default))
@@
     (stroke (width 0) (type default))
   )
-  (wire (pts (xy 262.255 54.61) (xy 267.335 54.61))
-    (stroke (width 0) (type default))
-  )
   (wire (pts (xy 45.72 97.155) (xy 54.61 97.155))
     (stroke (width 0) (type default))
@@
     (stroke (width 0) (type default))
   )
-  (wire (pts (xy 254 47.625) (xy 262.255 47.625))
-    (stroke (width 0) (type default))
-  )
   (wire (pts (xy 258.445 135.255) (xy 260.985 135.255))
     (stroke (width 0) (type default))
@@
     (stroke (width 0) (type default))
   )
-  (wire (pts (xy 262.255 47.625) (xy 262.255 54.61))
-    (stroke (width 0) (type default))
-  )
   (wire (pts (xy 169.545 139.065) (xy 182.88 139.065))
     (stroke (width 0) (type default))
@@
     (stroke (width 0) (type default))
   )
+  (wire (pts (xy 256.54 54.61) (xy 267.335 54.61))
+    (stroke (width 0) (type default))
+  )
   (wire (pts (xy 247.65 160.655) (xy 254 160.655))
     (stroke (width 0) (type default))
@@
       (effects (font (size 1.27 1.27)) (justify right))
     )
-    (property "Footprint" "Capacitor_THT:C_Rect_L10.0mm_W4.0mm_P7.50mm_MKS4" (at 66.9798 67.31 0)
+    (property "Footprint" "Capacitor_THT:C_Rect_L11.5mm_W5.6mm_P10.00mm_MKT" (at 66.9798 67.31 0)
       (effects (font (size 1.27 1.27)) hide)
     )
@@
       (effects (font (size 1.27 1.27)) hide)
     )
-    (property "LCSC#" "C2895620" (at 67.945 71.12 0)
+    (property "LCSC#" "C506867" (at 67.945 71.12 0)
       (effects (font (size 1.27 1.27)) hide)
     )
-    (property "Mouser#" "667-ECW-FD2J104K4" (at 67.945 71.12 0)
+    (property "Mouser#" "" (at 67.945 71.12 0)
       (effects (font (size 1.27 1.27)) hide)
     )
@@
       (effects (font (size 1.27 1.27)) hide)
     )
+    (property "LCSC#" "C255812" (at 272.415 54.61 0)
+      (effects (font (size 1.27 1.27)) hide)
+    )
+    (property "Mouser#" "179-TS046655BK160SMT" (at 272.415 54.61 0)
+      (effects (font (size 1.27 1.27)) hide)
+    )

Commit message: Mise a jour resistance puissance LED
Parts:
- R23: value 100R -> 330R
Other:
- note added: "2mA"
- note added: "7mA"
Changed lines of the file:
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@@
     (stroke (width 0) (type default))
+  )
+  (text "7mA" (at 76.2 48.895 0)
+    (effects (font (size 1 1)) (justify left bottom))
   )
   (text "MCP23017" (at 13.335 88.9 0)
@@
   (text "Relai" (at 14.605 17.78 0)
     (effects (font (size 2.2 2.2)) (justify left bottom))
+  )
+  (text "2mA" (at 241.935 163.83 0)
+    (effects (font (size 1 1)) (justify left bottom))
   )
   (text "Écran OLED" (at 160.655 76.835 0)
@@
       (effects (font (size 1.27 1.27)))
     )
-    (property "Value" "100R" (at 229.87 158.115 90)
-      (effects (font (size 1.27 1.27)))
-    )
+    (property "Value" "330R" (at 229.87 158.115 90)
+      (effects (font (size 1.27 1.27)))
+    )

Commit message: Mise a jour 1er assemblage
Parts:
- R23: LCSC# C17408 -> C105878; Mouser# 603-RC0805FR-07100RL -> 603-RC0805FR-07330RL
Changed lines of the file:
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@@
       (effects (font (size 1.27 1.27)) hide)
     )
-    (property "LCSC#" "C17408" (at 229.87 160.655 0)
+    (property "LCSC#" "C105878" (at 229.87 160.655 0)
       (effects (font (size 1.27 1.27)) hide)
     )
-    (property "Mouser#" "603-RC0805FR-07100RL" (at 229.87 160.655 0)
+    (property "Mouser#" "603-RC0805FR-07330RL" (at 229.87 160.655 0)
       (effects (font (size 1.27 1.27)) hide)
     )

Commit message: Fix transistor relai (collecteur et émeteur intervertis)
Connections:
- net GND: now also Q1.2 (E); no longer Q1.3 (C)
- net RL_TE: now also Q1.3 (C); no longer Q1.2 (E)
Other:
- moved on the sheet: Q1
Changed lines of the file:
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@@
     )
   )
-  (symbol (lib_id "remora_lib:MMBT2222") (at 56.515 38.735 270) (unit 1)
-    (in_bom yes) (on_board yes) (dnp no) (fields_autoplaced)
+  (symbol (lib_id "remora_lib:MMBT2222") (at 56.515 38.735 90) (mirror x) (unit 1)
+    (in_bom yes) (on_board yes) (dnp no)
     (property "Reference" "Q1" (at 56.515 45.085 90)
       (effects (font (size 1.27 1.27)))
@@
       (effects (font (size 1.27 1.27)))
     )
-    (property "Footprint" "Package_TO_SOT_SMD:SOT-23" (at 54.61 43.815 0)
+    (property "Footprint" "Package_TO_SOT_SMD:SOT-23" (at 58.42 43.815 0)
       (effects (font (size 1.27 1.27) italic) (justify left) hide)
     )

Commit message: Deplacement du pin teleinfo de SD1 à GPIO13
Connections:
- net TELEINFO: now also U16.29 (IO13/TCK); no longer U16.9 (SD1/SDI)
- no-connect marks 23 -> 22
Other:
- moved on the sheet: R21, R22, SW1, U16

Commit message: Nouvelles empreintes pour les diodes
Les pads des diodes ont été agrandies et espacées pour respecter la datasheet.
Changement ref des borniers pour du 2.5mm²
Parts:
- D1, D10, D11, D12, D13, D14, D15, D2, D3, D4, D5, D6, D7, D8, D9: footprint Diode_SMD:D_SOD-123F -> remora_lib:D_SOD-123FL
- J1: LCSC# C5188441 -> C5188464
- J2, J3, J4, J5, J6, J9: LCSC# C5188440 -> C5188463
Changed lines of the file:
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@@
 			)
 		)
-		(property "Footprint" "Diode_SMD:D_SOD-123F"
+		(property "Footprint" "remora_lib:D_SOD-123FL"
 			(at 146.05 106.045 0)
 			(effects
@@
 			)
 		)
-		(property "LCSC#" "C5188440"
+		(property "LCSC#" "C5188463"
 			(at 176.53 28.575 0)
 			(effects
@@
 			)
 		)
-		(property "Footprint" "Diode_SMD:D_SOD-123F"
+		(property "Footprint" "remora_lib:D_SOD-123FL"
 			(at 146.05 163.195 0)
 			(effects
@@
 			)
 		)
-		(property "LCSC#" "C5188440"
+		(property "LCSC#" "C5188463"
 			(at 176.53 40.005 0)
 			(effects
@@
 			)
 		)
-		(property "Footprint" "Diode_SMD:D_SOD-123F"
+		(property "Footprint" "remora_lib:D_SOD-123FL"
 			(at 37.465 30.48 0)
 			(effects
@@
 			)
 		)
-		(property "Footprint" "Diode_SMD:D_SOD-123F"
+		(property "Footprint" "remora_lib:D_SOD-123FL"
 			(at 146.05 37.465 0)
 			(effects
@@
 			)
 		)
-		(property "LCSC#" "C5188440"
+		(property "LCSC#" "C5188463"
 			(at 176.53 62.865 0)
 			(effects
@@
 			)
 		)
-		(property "LCSC#" "C5188440"
+		(property "LCSC#" "C5188463"
 			(at 27.94 185.42 0)
 			(effects
@@
 			)
 		)
-		(property "Footprint" "Diode_SMD:D_SOD-123F"
+		(property "Footprint" "remora_lib:D_SOD-123FL"
 			(at 146.05 140.335 0)
 			(effects
@@
 			)
 		)
-		(property "LCSC#" "C5188440"
+		(property "LCSC#" "C5188463"
 			(at 176.53 51.435 0)
 			(effects
@@
 			)
 		)
-		(property "Footprint" "Diode_SMD:D_SOD-123F"
+		(property "Footprint" "remora_lib:D_SOD-123FL"
 			(at 146.05 71.755 0)
 			(effects
@@
 			)
 		)
-		(property "Footprint" "Diode_SMD:D_SOD-123F"
+		(property "Footprint" "remora_lib:D_SOD-123FL"
 			(at 146.05 83.185 0)
 			(effects
@@
 			)
 		)
-		(property "Footprint" "Diode_SMD:D_SOD-123F"
+		(property "Footprint" "remora_lib:D_SOD-123FL"
 			(at 146.05 60.325 0)
 			(effects
@@
 			)
 		)
-		(property "Footprint" "Diode_SMD:D_SOD-123F"
+		(property "Footprint" "remora_lib:D_SOD-123FL"
 			(at 146.05 174.625 0)
 			(effects
@@
 			)
 		)
-		(property "Footprint" "Diode_SMD:D_SOD-123F"
+		(property "Footprint" "remora_lib:D_SOD-123FL"
 			(at 146.05 186.055 0)
 			(effects
@@
 			)
 		)
-		(property "LCSC#" "C5188441"
+		(property "LCSC#" "C5188464"
 			(at 31.115 69.85 0)
 			(effects
@@
 			)
 		)
-		(property "Footprint" "Diode_SMD:D_SOD-123F"
+		(property "Footprint" "remora_lib:D_SOD-123FL"
 			(at 146.05 151.765 0)
 			(effects
@@
 			)
 		)
-		(property "Footprint" "Diode_SMD:D_SOD-123F"
+		(property "Footprint" "remora_lib:D_SOD-123FL"
 			(at 146.05 117.475 0)
 			(effects
@@
 			)
 		)
-		(property "Footprint" "Diode_SMD:D_SOD-123F"
+		(property "Footprint" "remora_lib:D_SOD-123FL"
 			(at 146.05 48.895 0)
 			(effects
@@
 			)
 		)
-		(property "Footprint" "Diode_SMD:D_SOD-123F"
+		(property "Footprint" "remora_lib:D_SOD-123FL"
 			(at 146.05 94.615 0)
 			(effects
@@
 			)
 		)
-		(property "LCSC#" "C5188440"
+		(property "LCSC#" "C5188463"
 			(at 225.425 130.175 0)
 			(effects
@@
 			)
 		)
-		(property "Footprint" "Diode_SMD:D_SOD-123F"
+		(property "Footprint" "remora_lib:D_SOD-123FL"
 			(at 146.05 128.905 0)
 			(effects
